Commit message: Add waist joints to mock ros2_control configs for demo.launch.py
upper_body_controller drives waist + both arms, but the mock
(GenericSystem) ros2_control xacros used by demo.launch.py had no waist
joints, so the controller could not be activated. Add the three waist
joints to every variant.

Co-Authored-By: Claude Opus 5.5 <noreply@anthropic.com>
Claude-Session: https://claude.ai/code/session_01BUyB895TbRfCK2opkghDxb

File: g1_moveit_config/config/g1_29dof_with_hand.ros2_control.xacro (robot description, xacro)
@@ -8,4 +8,26 @@
         <plugin>mock_components/GenericSystem</plugin>
       </hardware>
+      <!-- Waist joints -->
+      <joint name="waist_yaw_joint">
+        <command_interface name="position"/>
+        <state_interface name="position">
+          <param name="initial_value">${initial_positions['waist_yaw_joint']}</param>
+        </state_interface>
+        <state_interface name="velocity"/>
+      </joint>
+      <joint name="waist_roll_joint">
+        <command_interface name="position"/>
+        <state_interface name="position">
+          <param name="initial_value">${initial_positions['waist_roll_joint']}</param>
+        </state_interface>
+        <state_interface name="velocity"/>
+      </joint>
+      <joint name="waist_pitch_joint">
+        <command_interface name="position"/>
+        <state_interface name="position">
+          <param name="initial_value">${initial_positions['waist_pitch_joint']}</param>
+        </state_interface>
+        <state_interface name="velocity"/>
+      </joint>
       <!-- Left arm joints -->
       <joint name="left_shoulder_pitch_joint">

File: g1_moveit_config/config/g1_inspire_dfq.ros2_control.xacro (robot description, xacro)
@@ -9,4 +9,26 @@
         <plugin>mock_components/GenericSystem</plugin>
       </hardware>
+      <!-- Waist joints -->
+      <joint name="waist_yaw_joint">
+        <command_interface name="position"/>
+        <state_interface name="position">
+          <param name="initial_value">${initial_positions['waist_yaw_joint']}</param>
+        </state_interface>
+        <state_interface name="velocity"/>
+      </joint>
+      <joint name="waist_roll_joint">
+        <command_interface name="position"/>
+        <state_interface name="position">
+          <param name="initial_value">${initial_positions['waist_roll_joint']}</param>
+        </state_interface>
+        <state_interface name="velocity"/>
+      </joint>
+      <joint name="waist_pitch_joint">
+        <command_interface name="position"/>
+        <state_interface name="position">
+          <param name="initial_value">${initial_positions['waist_pitch_joint']}</param>
+        </state_interface>
+        <state_interface name="velocity"/>
+      </joint>
       <!-- Left arm joints -->
       <joint name="left_shoulder_pitch_joint">

File: g1_moveit_config/config/g1_inspire_ftp.ros2_control.xacro (robot description, xacro)
@@ -9,4 +9,26 @@
         <plugin>mock_components/GenericSystem</plugin>
       </hardware>
+      <!-- Waist joints -->
+      <joint name="waist_yaw_joint">
+        <command_interface name="position"/>
+        <state_interface name="position">
+          <param name="initial_value">${initial_positions['waist_yaw_joint']}</param>
+        </state_interface>
+        <state_interface name="velocity"/>
+      </joint>
+      <joint name="waist_roll_joint">
+        <command_interface name="position"/>
+        <state_interface name="position">
+          <param name="initial_value">${initial_positions['waist_roll_joint']}</param>
+        </state_interface>
+        <state_interface name="velocity"/>
+      </joint>
+      <joint name="waist_pitch_joint">
+        <command_interface name="position"/>
+        <state_interface name="position">
+          <param name="initial_value">${initial_positions['waist_pitch_joint']}</param>
+        </state_interface>
+        <state_interface name="velocity"/>
+      </joint>
       <!-- Left arm joints -->
       <joint name="left_shoulder_pitch_joint">

File: g1_moveit_config/config/g1_no_hand.ros2_control.xacro (robot description, xacro)
@@ -7,4 +7,26 @@
         <plugin>mock_components/GenericSystem</plugin>
       </hardware>
+      <!-- Waist joints -->
+      <joint name="waist_yaw_joint">
+        <command_interface name="position"/>
+        <state_interface name="position">
+          <param name="initial_value">${initial_positions['waist_yaw_joint']}</param>
+        </state_interface>
+        <state_interface name="velocity"/>
+      </joint>
+      <joint name="waist_roll_joint">
+        <command_interface name="position"/>
+        <state_interface name="position">
+          <param name="initial_value">${initial_positions['waist_roll_joint']}</param>
+        </state_interface>
+        <state_interface name="velocity"/>
+      </joint>
+      <joint name="waist_pitch_joint">
+        <command_interface name="position"/>
+        <state_interface name="position">
+          <param name="initial_value">${initial_positions['waist_pitch_joint']}</param>
+        </state_interface>
+        <state_interface name="velocity"/>
+      </joint>
       <!-- Left arm joints -->
       <joint name="left_shoulder_pitch_joint">
